File: ES9033_prototype/LDO_LT3042_3v3.kicad_sch (KiCad schematic)
At the start: 7 parts, among them U301 LT3042

Commit message: added schematic title
Other:
- company: (none) -> Fabian Muehlberger 
- title: (none) -> ES9033 DAC prototype
Changed lines of the file:
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@@
 (kicad_sch (version 20211123) (generator eeschema)
   (paper "A4")
+  (title_block
+    (title "ES9033 DAC prototype")
+    (date "2022-09-09")
+    (rev "0.1")
+    (company "Fabian Muehlberger ")
+  )
   (junction (at 118.11 64.77) (diameter 0) (color 0 0 0 0)
   )
